File: V1/eumesmo-rl-4ch12a-nc-v1.kicad_pcb (KiCad board)
At the start: 2 copper layers, 68 x 67.8 mm, 25 parts, among them J1 250-202, J2 250-204, J3 DB142V-5.08-4P, J4 DB142V-5.08-4P, K1 Songle_SRD_1B, K2 Songle_SRD_1B, K3 Songle_SRD_1B, K4 Songle_SRD_1B

Commit message: Renamed all files to the eumesmo branding
Other:
- board text added: "eumesmo-rl-4ch12a-nc"
- board text removed: "RELAY-24V-4CH-12A-NC-V1"
Changed lines of the file:
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@@
 		(property ki_fp_filters "R_*")
 		(sheetname "/")
-		(sheetfile "relay-24v-4ch-12a-nc-v1.kicad_sch")
+		(sheetfile "eumesmo-rl-4ch12a-nc.kicad_sch")
 		(units
 			(unit
@@
 		(property ki_fp_filters "Connector*:*_1x??_*")
 		(sheetname "/")
-		(sheetfile "relay-24v-4ch-12a-nc-v1.kicad_sch")
+		(sheetfile "eumesmo-rl-4ch12a-nc.kicad_sch")
 		(units
 			(unit
@@
 		(property ki_fp_filters "TO-???* *_Diode_* *SingleDiode* D_*")
 		(sheetname "/")
-		(sheetfile "relay-24v-4ch-12a-nc-v1.kicad_sch")
+		(sheetfile "eumesmo-rl-4ch12a-nc.kicad_sch")
 		(units
 			(unit
@@
 		(property ki_fp_filters "LED* LED_SMD:* LED_THT:*")
 		(sheetname "/")
-		(sheetfile "relay-24v-4ch-12a-nc-v1.kicad_sch")
+		(sheetfile "eumesmo-rl-4ch12a-nc.kicad_sch")
 		(units
 			(unit
@@
 		(property ki_fp_filters "Connector*:*_1x??_*")
 		(sheetname "/")
-		(sheetfile "relay-24v-4ch-12a-nc-v1.kicad_sch")
+		(sheetfile "eumesmo-rl-4ch12a-nc.kicad_sch")
 		(units
 			(unit
@@
 		(property ki_fp_filters "R_*")
 		(sheetname "/")
-		(sheetfile "relay-24v-4ch-12a-nc-v1.kicad_sch")
+		(sheetfile "eumesmo-rl-4ch12a-nc.kicad_sch")
 		(units
 			(unit
@@
 		(property ki_fp_filters "LED* LED_SMD:* LED_THT:*")
 		(sheetname "/")
-		(sheetfile "relay-24v-4ch-12a-nc-v1.kicad_sch")
+		(sheetfile "eumesmo-rl-4ch12a-nc.kicad_sch")
 		(units
 			(unit
@@
 		(property ki_fp_filters "R_*")
 		(sheetname "/")
-		(sheetfile "relay-24v-4ch-12a-nc-v1.kicad_sch")
+		(sheetfile "eumesmo-rl-4ch12a-nc.kicad_sch")
 		(units
 			(unit
@@
 		(property ki_fp_filters "TO-???* *_Diode_* *SingleDiode* D_*")
 		(sheetname "/")
-		(sheetfile "relay-24v-4ch-12a-nc-v1.kicad_sch")
+		(sheetfile "eumesmo-rl-4ch12a-nc.kicad_sch")
 		(units
 			(unit
@@
 		(property ki_fp_filters "Relay*SPDT*Finder*40.11*")
 		(sheetname "/")
-		(sheetfile "relay-24v-4ch-12a-nc-v1.kicad_sch")
+		(sheetfile "eumesmo-rl-4ch12a-nc.kicad_sch")
 		(units
 			(unit
@@
 		(property ki_fp_filters "RV_* Varistor*")
 		(sheetname "/")
-		(sheetfile "relay-24v-4ch-12a-nc-v1.kicad_sch")
+		(sheetfile "eumesmo-rl-4ch12a-nc.kicad_sch")
 		(units
 			(unit
@@
 		(property ki_fp_filters "Relay*SPDT*Finder*40.11*")
 		(sheetname "/")
-		(sheetfile "relay-24v-4ch-12a-nc-v1.kicad_sch")
+		(sheetfile "eumesmo-rl-4ch12a-nc.kicad_sch")
 		(units
 			(unit
@@
 		(property ki_fp_filters "Relay*SPDT*Finder*40.11*")
 		(sheetname "/")
-		(sheetfile "relay-24v-4ch-12a-nc-v1.kicad_sch")
+		(sheetfile "eumesmo-rl-4ch12a-nc.kicad_sch")
 		(units
 			(unit
@@
 		(property ki_fp_filters "TO-???* *_Diode_* *SingleDiode* D_*")
 		(sheetname "/")
-		(sheetfile "relay-24v-4ch-12a-nc-v1.kicad_sch")
+		(sheetfile "eumesmo-rl-4ch12a-nc.kicad_sch")
 		(units
 			(unit
@@
 		(property ki_fp_filters "Connector*:*_1x??_*")
 		(sheetname "/")
-		(sheetfile "relay-24v-4ch-12a-nc-v1.kicad_sch")
+		(sheetfile "eumesmo-rl-4ch12a-nc.kicad_sch")
 		(units
 			(unit
@@
 		(property ki_fp_filters "LED* LED_SMD:* LED_THT:*")
 		(sheetname "/")
-		(sheetfile "relay-24v-4ch-12a-nc-v1.kicad_sch")
+		(sheetfile "eumesmo-rl-4ch12a-nc.kicad_sch")
 		(units
 			(unit
@@
 		(property ki_fp_filters "RV_* Varistor*")
 		(sheetname "/")
-		(sheetfile "relay-24v-4ch-12a-nc-v1.kicad_sch")
+		(sheetfile "eumesmo-rl-4ch12a-nc.kicad_sch")
 		(units
 			(unit
@@
 		(property ki_fp_filters "RV_* Varistor*")
 		(sheetname "/")
-		(sheetfile "relay-24v-4ch-12a-nc-v1.kicad_sch")
+		(sheetfile "eumesmo-rl-4ch12a-nc.kicad_sch")
 		(units
 			(unit
@@
 		(property ki_fp_filters "Connector*:*_1x??_*")
 		(sheetname "/")
-		(sheetfile "relay-24v-4ch-12a-nc-v1.kicad_sch")
+		(sheetfile "eumesmo-rl-4ch12a-nc.kicad_sch")
 		(units
 			(unit
@@
 		(property ki_fp_filters "TO-???* *_Diode_* *SingleDiode* D_*")
 		(sheetname "/")
-		(sheetfile "relay-24v-4ch-12a-nc-v1.kicad_sch")
+		(sheetfile "eumesmo-rl-4ch12a-nc.kicad_sch")
 		(units
 			(unit
@@
 		(property ki_fp_filters "RV_* Varistor*")
 		(sheetname "/")
-		(sheetfile "relay-24v-4ch-12a-nc-v1.kicad_sch")
+		(sheetfile "eumesmo-rl-4ch12a-nc.kicad_sch")
 		(units
 			(unit
@@
 		(property ki_fp_filters "R_*")
 		(sheetname "/")
-		(sheetfile "relay-24v-4ch-12a-nc-v1.kicad_sch")
+		(sheetfile "eumesmo-rl-4ch12a-nc.kicad_sch")
 		(units
 			(unit
@@
 		(property ki_fp_filters "Relay*SPDT*Finder*40.11*")
 		(sheetname "/")
-		(sheetfile "relay-24v-4ch-12a-nc-v1.kicad_sch")
+		(sheetfile "eumesmo-rl-4ch12a-nc.kicad_sch")
 		(units
 			(unit
@@
 		(property ki_fp_filters "LED* LED_SMD:* LED_THT:*")
 		(sheetname "/")
-		(sheetfile "relay-24v-4ch-12a-nc-v1.kicad_sch")
+		(sheetfile "eumesmo-rl-4ch12a-nc.kicad_sch")
 		(units
 			(unit
@@
 		)
 	)
-	(gr_text "RELAY-24V-4CH-12A-NC-V1"
+	(gr_text "eumesmo-rl-4ch12a-nc"
 		(at 141.5 64.5 0)
 		(layer "F.SilkS")

Commit message: Adjusted PCB version number.
Changed lines of the file:
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@@
 	(paper "A4")
 	(title_block
-		(title "4x 24V Relay Module with NC contacts")
-		(date "2026-06-11")
-		(rev "V1.1")
+		(title "eumesmo 4x 24V Relay Module with NC contacts")
+		(date "2026-06-13")
+		(rev "V1.2")
 	)
 	(layers
@@
 			(font
 				(size 1.5 1.1)
-				(thickness 0.25)
+				(thickness 0.2)
 				(bold yes)
 			)

Commit message: Renamed all files to eumesmo branding
Other:
- board text added: "V1.2 2026-06-13"
- board text removed: "V1.1 2026-06-12"
Changed lines of the file:
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@@
 		(layer "Edge.Cuts")
 	)
-	(gr_text "V1.1\n2026-06-12"
+	(gr_text "V1.2\n2026-06-13"
 		(at 162.75 117.625 0)
 		(layer "F.SilkS")

Commit message: Release V1.2.0
Other:
- board text added: "V1.2 2026-06-17"
- board text removed: "V1.2 2026-06-13"
Changed lines of the file:
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@@
 		(property ki_fp_filters "R_*")
 		(sheetname "/")
-		(sheetfile "eumesmo-rl-4ch12a-nc.kicad_sch")
+		(sheetfile "eumesmo-rl-4ch12a-nc-v1.kicad_sch")
 		(units
 			(unit
@@
 		(property ki_fp_filters "Connector*:*_1x??_*")
 		(sheetname "/")
-		(sheetfile "eumesmo-rl-4ch12a-nc.kicad_sch")
+		(sheetfile "eumesmo-rl-4ch12a-nc-v1.kicad_sch")
 		(units
 			(unit
@@
 		(property ki_fp_filters "TO-???* *_Diode_* *SingleDiode* D_*")
 		(sheetname "/")
-		(sheetfile "eumesmo-rl-4ch12a-nc.kicad_sch")
+		(sheetfile "eumesmo-rl-4ch12a-nc-v1.kicad_sch")
 		(units
 			(unit
@@
 		(property ki_fp_filters "LED* LED_SMD:* LED_THT:*")
 		(sheetname "/")
-		(sheetfile "eumesmo-rl-4ch12a-nc.kicad_sch")
+		(sheetfile "eumesmo-rl-4ch12a-nc-v1.kicad_sch")
 		(units
 			(unit
@@
 		(property ki_fp_filters "Connector*:*_1x??_*")
 		(sheetname "/")
-		(sheetfile "eumesmo-rl-4ch12a-nc.kicad_sch")
+		(sheetfile "eumesmo-rl-4ch12a-nc-v1.kicad_sch")
 		(units
 			(unit
@@
 		(property ki_fp_filters "R_*")
 		(sheetname "/")
-		(sheetfile "eumesmo-rl-4ch12a-nc.kicad_sch")
+		(sheetfile "eumesmo-rl-4ch12a-nc-v1.kicad_sch")
 		(units
 			(unit
@@
 		(property ki_fp_filters "LED* LED_SMD:* LED_THT:*")
 		(sheetname "/")
-		(sheetfile "eumesmo-rl-4ch12a-nc.kicad_sch")
+		(sheetfile "eumesmo-rl-4ch12a-nc-v1.kicad_sch")
 		(units
 			(unit
@@
 		(property ki_fp_filters "R_*")
 		(sheetname "/")
-		(sheetfile "eumesmo-rl-4ch12a-nc.kicad_sch")
+		(sheetfile "eumesmo-rl-4ch12a-nc-v1.kicad_sch")
 		(units
 			(unit
@@
 		(property ki_fp_filters "TO-???* *_Diode_* *SingleDiode* D_*")
 		(sheetname "/")
-		(sheetfile "eumesmo-rl-4ch12a-nc.kicad_sch")
+		(sheetfile "eumesmo-rl-4ch12a-nc-v1.kicad_sch")
 		(units
 			(unit
@@
 		(property ki_fp_filters "Relay*SPDT*Finder*40.11*")
 		(sheetname "/")
-		(sheetfile "eumesmo-rl-4ch12a-nc.kicad_sch")
+		(sheetfile "eumesmo-rl-4ch12a-nc-v1.kicad_sch")
 		(units
 			(unit
@@
 		(property ki_fp_filters "RV_* Varistor*")
 		(sheetname "/")
-		(sheetfile "eumesmo-rl-4ch12a-nc.kicad_sch")
+		(sheetfile "eumesmo-rl-4ch12a-nc-v1.kicad_sch")
 		(units
 			(unit
@@
 		(property ki_fp_filters "Relay*SPDT*Finder*40.11*")
 		(sheetname "/")
-		(sheetfile "eumesmo-rl-4ch12a-nc.kicad_sch")
+		(sheetfile "eumesmo-rl-4ch12a-nc-v1.kicad_sch")
 		(units
 			(unit
@@
 		(property ki_fp_filters "Relay*SPDT*Finder*40.11*")
 		(sheetname "/")
-		(sheetfile "eumesmo-rl-4ch12a-nc.kicad_sch")
+		(sheetfile "eumesmo-rl-4ch12a-nc-v1.kicad_sch")
 		(units
 			(unit
@@
 		(property ki_fp_filters "TO-???* *_Diode_* *SingleDiode* D_*")
 		(sheetname "/")
-		(sheetfile "eumesmo-rl-4ch12a-nc.kicad_sch")
+		(sheetfile "eumesmo-rl-4ch12a-nc-v1.kicad_sch")
 		(units
 			(unit
@@
 		(property ki_fp_filters "Connector*:*_1x??_*")
 		(sheetname "/")
-		(sheetfile "eumesmo-rl-4ch12a-nc.kicad_sch")
+		(sheetfile "eumesmo-rl-4ch12a-nc-v1.kicad_sch")
 		(units
 			(unit
@@
 		(property ki_fp_filters "LED* LED_SMD:* LED_THT:*")
 		(sheetname "/")
-		(sheetfile "eumesmo-rl-4ch12a-nc.kicad_sch")
+		(sheetfile "eumesmo-rl-4ch12a-nc-v1.kicad_sch")
 		(units
 			(unit
@@
 		(property ki_fp_filters "RV_* Varistor*")
 		(sheetname "/")
-		(sheetfile "eumesmo-rl-4ch12a-nc.kicad_sch")
+		(sheetfile "eumesmo-rl-4ch12a-nc-v1.kicad_sch")
 		(units
 			(unit
@@
 		(property ki_fp_filters "RV_* Varistor*")
 		(sheetname "/")
-		(sheetfile "eumesmo-rl-4ch12a-nc.kicad_sch")
+		(sheetfile "eumesmo-rl-4ch12a-nc-v1.kicad_sch")
 		(units
 			(unit
@@
 		(property ki_fp_filters "Connector*:*_1x??_*")
 		(sheetname "/")
-		(sheetfile "eumesmo-rl-4ch12a-nc.kicad_sch")
+		(sheetfile "eumesmo-rl-4ch12a-nc-v1.kicad_sch")
 		(units
 			(unit
@@
 		(property ki_fp_filters "TO-???* *_Diode_* *SingleDiode* D_*")
 		(sheetname "/")
-		(sheetfile "eumesmo-rl-4ch12a-nc.kicad_sch")
+		(sheetfile "eumesmo-rl-4ch12a-nc-v1.kicad_sch")
 		(units
 			(unit
@@
 		(property ki_fp_filters "RV_* Varistor*")
 		(sheetname "/")
-		(sheetfile "eumesmo-rl-4ch12a-nc.kicad_sch")
+		(sheetfile "eumesmo-rl-4ch12a-nc-v1.kicad_sch")
 		(units
 			(unit
@@
 		(property ki_fp_filters "R_*")
 		(sheetname "/")
-		(sheetfile "eumesmo-rl-4ch12a-nc.kicad_sch")
+		(sheetfile "eumesmo-rl-4ch12a-nc-v1.kicad_sch")
 		(units
 			(unit
@@
 		(property ki_fp_filters "Relay*SPDT*Finder*40.11*")
 		(sheetname "/")
-		(sheetfile "eumesmo-rl-4ch12a-nc.kicad_sch")
+		(sheetfile "eumesmo-rl-4ch12a-nc-v1.kicad_sch")
 		(units
 			(unit
@@
 		(property ki_fp_filters "LED* LED_SMD:* LED_THT:*")
 		(sheetname "/")
-		(sheetfile "eumesmo-rl-4ch12a-nc.kicad_sch")
+		(sheetfile "eumesmo-rl-4ch12a-nc-v1.kicad_sch")
 		(units
 			(unit
@@
 		)
 	)
+	(gr_rect
+		(start 126.5 126)
+		(end 134 127.5)
+		(stroke
+			(width 0.1)
+			(type solid)
+		)
+		(fill no)
+		(layer "F.SilkS")
+	)
 	(gr_line
 		(start 131 69)
@@
 	)
 	(gr_rect
-		(start 160 116.375)
-		(end 165.5 119.125)
-		(stroke
-			(width 0.1)
-			(type solid)
-		)
-		(fill no)
-		(layer "F.SilkS")
-	)
-	(gr_rect
 		(start 166 62.75)
 		(end 180 64.75)
@@
 		(layer "Edge.Cuts")
 	)
-	(gr_text "V1.2\n2026-06-13"
-		(at 162.75 117.625 0)
+	(gr_text "V1.2 2026-06-17"
+		(at 130.25 126.75 0)
 		(layer "F.SilkS")
 		(effects
