File: V1/eumesmo-rl-4ch12a-nc-v1.kicad_sch (KiCad schematic)
At the start: 24 parts, among them J1 250-202, J2 250-204, J3 DB142V-5.08-4P, J4 DB142V-5.08-4P, K1 Songle_SRD_1B, K2 Songle_SRD_1B, K3 Songle_SRD_1B, K4 Songle_SRD_1B

Commit message: Adjusted PCB version number.
Other:
- title: 4x 24V Relay Module -> eumesmo 4x 24V Relay Module
Changed lines of the file:
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@@
 	(paper "A4")
 	(title_block
-		(title "4x 24V Relay Module")
-		(date "2026-06-11")
-		(rev "V1.1")
+		(title "eumesmo 4x 24V Relay Module")
+		(date "2026-06-13")
+		(rev "V1.2")
 	)
 	(junction
@@
 		)
 		(instances
-			(project "eumesmo-rl-4ch12a-nc"
+			(project "eumesmo-rl-4ch12a-nc-v1"
 				(path "/57cfb5e7-a9ab-4784-80b3-e51e693f5cc8"
 					(reference "#PWR0103")
@@
 		)
 		(instances
-			(project "eumesmo-rl-4ch12a-nc"
+			(project "eumesmo-rl-4ch12a-nc-v1"
 				(path "/57cfb5e7-a9ab-4784-80b3-e51e693f5cc8"
 					(reference "D7")
@@
 		)
 		(instances
-			(project "eumesmo-rl-4ch12a-nc"
+			(project "eumesmo-rl-4ch12a-nc-v1"
 				(path "/57cfb5e7-a9ab-4784-80b3-e51e693f5cc8"
 					(reference "D2")
@@
 		)
 		(instances
-			(project "eumesmo-rl-4ch12a-nc"
+			(project "eumesmo-rl-4ch12a-nc-v1"
 				(path "/57cfb5e7-a9ab-4784-80b3-e51e693f5cc8"
 					(reference "K3")
@@
 		)
 		(instances
-			(project "eumesmo-rl-4ch12a-nc"
+			(project "eumesmo-rl-4ch12a-nc-v1"
 				(path "/57cfb5e7-a9ab-4784-80b3-e51e693f5cc8"
 					(reference "J2")
@@
 		)
 		(instances
-			(project "eumesmo-rl-4ch12a-nc"
+			(project "eumesmo-rl-4ch12a-nc-v1"
 				(path "/57cfb5e7-a9ab-4784-80b3-e51e693f5cc8"
 					(reference "K2")
@@
 		)
 		(instances
-			(project "eumesmo-rl-4ch12a-nc"
+			(project "eumesmo-rl-4ch12a-nc-v1"
 				(path "/57cfb5e7-a9ab-4784-80b3-e51e693f5cc8"
 					(reference "R1")
@@
 		)
 		(instances
-			(project "eumesmo-rl-4ch12a-nc"
+			(project "eumesmo-rl-4ch12a-nc-v1"
 				(path "/57cfb5e7-a9ab-4784-80b3-e51e693f5cc8"
 					(reference "#PWR0101")
@@
 		)
 		(instances
-			(project "eumesmo-rl-4ch12a-nc"
+			(project "eumesmo-rl-4ch12a-nc-v1"
 				(path "/57cfb5e7-a9ab-4784-80b3-e51e693f5cc8"
 					(reference "#FLG0101")
@@
 		)
 		(instances
-			(project "eumesmo-rl-4ch12a-nc"
+			(project "eumesmo-rl-4ch12a-nc-v1"
 				(path "/57cfb5e7-a9ab-4784-80b3-e51e693f5cc8"
 					(reference "D5")
@@
 		)
 		(instances
-			(project "eumesmo-rl-4ch12a-nc"
+			(project "eumesmo-rl-4ch12a-nc-v1"
 				(path "/57cfb5e7-a9ab-4784-80b3-e51e693f5cc8"
 					(reference "R3")
@@
 		)
 		(instances
-			(project "eumesmo-rl-4ch12a-nc"
+			(project "eumesmo-rl-4ch12a-nc-v1"
 				(path "/57cfb5e7-a9ab-4784-80b3-e51e693f5cc8"
 					(reference "J1")
@@
 		)
 		(instances
-			(project "eumesmo-rl-4ch12a-nc"
+			(project "eumesmo-rl-4ch12a-nc-v1"
 				(path "/57cfb5e7-a9ab-4784-80b3-e51e693f5cc8"
 					(reference "J3")
@@
 		)
 		(instances
-			(project "eumesmo-rl-4ch12a-nc"
+			(project "eumesmo-rl-4ch12a-nc-v1"
 				(path "/57cfb5e7-a9ab-4784-80b3-e51e693f5cc8"
 					(reference "#PWR0105")
@@
 		)
 		(instances
-			(project "eumesmo-rl-4ch12a-nc"
+			(project "eumesmo-rl-4ch12a-nc-v1"
 				(path "/57cfb5e7-a9ab-4784-80b3-e51e693f5cc8"
 					(reference "RV4")
@@
 		)
 		(instances
-			(project "eumesmo-rl-4ch12a-nc"
+			(project "eumesmo-rl-4ch12a-nc-v1"
 				(path "/57cfb5e7-a9ab-4784-80b3-e51e693f5cc8"
 					(reference "R4")
@@
 		)
 		(instances
-			(project "eumesmo-rl-4ch12a-nc"
+			(project "eumesmo-rl-4ch12a-nc-v1"
 				(path "/57cfb5e7-a9ab-4784-80b3-e51e693f5cc8"
 					(reference "D1")
@@
 		)
 		(instances
-			(project "eumesmo-rl-4ch12a-nc"
+			(project "eumesmo-rl-4ch12a-nc-v1"
 				(path "/57cfb5e7-a9ab-4784-80b3-e51e693f5cc8"
 					(reference "RV2")
@@
 		)
 		(instances
-			(project "eumesmo-rl-4ch12a-nc"
+			(project "eumesmo-rl-4ch12a-nc-v1"
 				(path "/57cfb5e7-a9ab-4784-80b3-e51e693f5cc8"
 					(reference "J4")
@@
 		)
 		(instances
-			(project "eumesmo-rl-4ch12a-nc"
+			(project "eumesmo-rl-4ch12a-nc-v1"
 				(path "/57cfb5e7-a9ab-4784-80b3-e51e693f5cc8"
 					(reference "R2")
@@
 		)
 		(instances
-			(project "eumesmo-rl-4ch12a-nc"
+			(project "eumesmo-rl-4ch12a-nc-v1"
 				(path "/57cfb5e7-a9ab-4784-80b3-e51e693f5cc8"
 					(reference "#PWR0104")
@@
 		)
 		(instances
-			(project "eumesmo-rl-4ch12a-nc"
+			(project "eumesmo-rl-4ch12a-nc-v1"
 				(path "/57cfb5e7-a9ab-4784-80b3-e51e693f5cc8"
 					(reference "D8")
@@
 		)
 		(instances
-			(project "eumesmo-rl-4ch12a-nc"
+			(project "eumesmo-rl-4ch12a-nc-v1"
 				(path "/57cfb5e7-a9ab-4784-80b3-e51e693f5cc8"
 					(reference "#PWR0102")
@@
 		)
 		(instances
-			(project "eumesmo-rl-4ch12a-nc"
+			(project "eumesmo-rl-4ch12a-nc-v1"
 				(path "/57cfb5e7-a9ab-4784-80b3-e51e693f5cc8"
 					(reference "D6")
@@
 		)
 		(instances
-			(project "eumesmo-rl-4ch12a-nc"
+			(project "eumesmo-rl-4ch12a-nc-v1"
 				(path "/57cfb5e7-a9ab-4784-80b3-e51e693f5cc8"
 					(reference "D3")
@@
 		)
 		(instances
-			(project "eumesmo-rl-4ch12a-nc"
+			(project "eumesmo-rl-4ch12a-nc-v1"
 				(path "/57cfb5e7-a9ab-4784-80b3-e51e693f5cc8"
 					(reference "K4")
@@
 		)
 		(instances
-			(project "eumesmo-rl-4ch12a-nc"
+			(project "eumesmo-rl-4ch12a-nc-v1"
 				(path "/57cfb5e7-a9ab-4784-80b3-e51e693f5cc8"
 					(reference "D4")
@@
 		)
 		(instances
-			(project "eumesmo-rl-4ch12a-nc"
+			(project "eumesmo-rl-4ch12a-nc-v1"
 				(path "/57cfb5e7-a9ab-4784-80b3-e51e693f5cc8"
 					(reference "RV1")
@@
 		)
 		(instances
-			(project "eumesmo-rl-4ch12a-nc"
+			(project "eumesmo-rl-4ch12a-nc-v1"
 				(path "/57cfb5e7-a9ab-4784-80b3-e51e693f5cc8"
 					(reference "K1")
@@
 		)
 		(instances
-			(project "eumesmo-rl-4ch12a-nc"
+			(project "eumesmo-rl-4ch12a-nc-v1"
 				(path "/57cfb5e7-a9ab-4784-80b3-e51e693f5cc8"
 					(reference "RV3")
